File: RoboSumoV1.0/Sumo.kicad_sch (KiCad schematic)
At the start: 28 parts, among them J1 BAT, J10 Conn_01x04_Pin, J2 ICSP, J4 ICSP, J5 Conn_01x06_MountingPin, J6 MotB, J7 MotA, J8 Conn_01x03_Pin, J9 I2C_Sensors, SW1 SW_SPDT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

Commit message: f
Other:
- moved on the sheet: J1, J10, J2, J4, J5, J8, J9, SW1, SW3, U2
